File: ImageProc_2.5.sch (EAGLE design)
At the start: 50 parts, among them J2 MOLEX_5034800600, U1 MIC5335-SPYMT, U11 ANTENNA-CHIP, U2 MIC5320-JGYML, U3 AT45DB321D, U4 ITG-3200, U6 ECS-2033, U7 ECS-160-8, U8 AT86RF231-ZU, U9 MN13822-L

Commit message: Stopped committing for a week. Oops.
Parts:
- removed BALUN1: HHM1710D1, stan:BALUNA
- removed J2: MOLEX_5034800600, stan:MOLEX_5034800600
- removed LED4: Yellow, led:LEDCHIP-LED0603
- removed LED5: Green, led:LEDCHIP-LED0603
- removed LED6: Red, led:LEDCHIP-LED0603
- removed PROC1: DSPIC33FJ128MC706A, stan:DSPIC33FJ128MC706-I/PT
- removed U1: MIC5335-SPYMT, stan:MIC5320-JGYML
- removed U11: ANTENNA-CHIP, stan:ANTENNA-CHIP
- removed U2: MIC5320-JGYML, stan:MIC5320-JGYML
- removed U3: AT45DB321D, stan:AT45DB321D
- removed U4: ITG-3200, stan:ITG-3200-00
- removed U6: ECS-2033, stan:OSCILLATORS
- removed U7: ECS-160-8, stan:CRYSTALS
- removed U8: AT86RF231-ZU, stan:AT86RF231-ZU
- removed U9: MN13822-L, stan:VOL_DETECTOR
- added ANT1: ANT8030-2R4-01A, biomimetic:ANT8030-2R4-01A
- added B1: HHM1710D1, biomimetic:HHM1710D1
- added C10, C20, C22, C27, C36, C37, C39, C40, C9: 0.1uF, biomimetic:CAP0402-CAP
- added C18, C19: 10pF, biomimetic:CAP0402-CAP
- added C21: 1uF, biomimetic:CAP0402-CAP
- added C32, C35: 2.2uF, biomimetic:CAP0402-CAP
- added C33: 22uF, biomimetic:CAP0603-CAP
- added C34: 10nF, biomimetic:CAP0402-CAP
- added C38: 2.2nF, biomimetic:CAP0402-CAP
- added IC1: XC61GC3002HR-G, biomimetic:XC61GC3002HR-G
- added IC10: AT45DB642D-CNU, biomimetic:AT45DB642D-CNU
- added IC2: MIC5335-SPYMT, biomimetic:MIC5335-SPYMT
- added IC3: MIC5335-JGYMT, biomimetic:MIC5335-JGYMT
- added IC4: DSPIC33FJ128MC706A, biomimetic:DSPIC33FJ128MC706A
- added IC5: AT86RF233-ZU, biomimetic:AT86RF233-ZU
- added IC6: LTC6088, biomimetic:LTC6088
- added IC7, IC8: DRV8833RTY, biomimetic:DRV8833RTY
- added IC9: MPU-6000, biomimetic:MPU-6000
- added JP1: MOLEX_503480-0600, biomimetic:MOLEX_503480-0600
- added JP4: 51441-2493-C, biomimetic:OV7660FSL_CON
- added L1: 4.7uH, biomimetic:INDUCTOR0603
- added LED1: YELLOW, biomimetic:LED0603
- added LED2, LED_RX: GREEN, biomimetic:LED0603
- added LED3, LED_TX: RED, biomimetic:LED0603
- added OSC1: ECS-2033-400, biomimetic:ECS-2033-400
- added OSC2: NX2520SA-16.000000MHZ, biomimetic:NX2520SA-16.000000MHZ
- added P1: BAT+, wirepad:SMD2
- added P10: MD2, wirepad:SMD2
- added P11: EXT1, wirepad:SMD2
- added P12: EXT2, wirepad:SMD2
- added P13: EXT3, wirepad:SMD2
- added P14: EXT4, wirepad:SMD2
- added P15: EXT5, wirepad:SMD2
- added P16: EXT6, wirepad:SMD2
- added P2: BAT-, wirepad:SMD2
- added P3: MA1, wirepad:SMD2
- added P4: MA2, wirepad:SMD2
- added P5: MB1, wirepad:SMD2
- added P6: MB2, wirepad:SMD2
- added P7: MC1, wirepad:SMD2
- added P8: MC2, wirepad:SMD2
- added P9: MD1, wirepad:SMD2
- added R12, R15, R21, R22, R25, R8: 15k, biomimetic:RESISTOR0402-RES
- added R14, R19, R20, R23, R24, R9: 47k, biomimetic:RESISTOR0402-RES
- added R26, R27, R28, R6, R7: 2.7k, biomimetic:RESISTOR0402-RES
- added R5: 4.7k, biomimetic:RESISTOR0402-RES
- C1: value 2.2nF -> 1uF; device SparkFun:CAP0402-CAP -> biomimetic:CAP0402-CAP
- C11, C12, C13, C26: value 1uF -> 0.1uF; device SparkFun:CAP0402-CAP -> biomimetic:CAP0402-CAP
- C14: value 22pF -> 0.1uF; device SparkFun:CAP0402-CAP -> biomimetic:CAP0402-CAP
- C15: value 1uF -> 4.7uF; device SparkFun:CAP0402-CAP -> biomimetic:CAP0603-CAP; COMMENT (none) -> ESR < 5 Ohm; TECHNOLOGY (none) -> CERAMIC; VOLTAGE (none) -> 16V
- C16, C17: value 1uF -> 22pF; device SparkFun:CAP0402-CAP -> biomimetic:CAP0402-CAP; DIELECTRIC (none) -> C0G; TECHNOLOGY (none) -> CERAMIC; TOLERANCE (none) -> 5%; VOLTAGE (none) -> 50V
- C2, C3: device SparkFun:CAP0402-CAP -> biomimetic:CAP0402-CAP
- C23: value 0.1uF -> 1uF; device SparkFun:CAP0402-CAP -> biomimetic:CAP0402-CAP; DIELECTRIC (none) -> X5R; TECHNOLOGY (none) -> CERAMIC; TOLERANCE (none) -> 10%; VOLTAGE (none) -> 16V
- C24, C25: value 1uF -> 0.1uF; device SparkFun:CAP0402-CAP -> biomimetic:CAP0402-CAP; TECHNOLOGY (none) -> CERAMIC; VOLTAGE (none) -> 10V
- C28: value 22pF -> 0.1uF; device SparkFun:CAP0402-CAP -> biomimetic:CAP0402-CAP; TECHNOLOGY (none) -> CERAMIC; VOLTAGE (none) -> 10V
- C29: value 12pF -> 0.1uF; device SparkFun:CAP0402-CAP -> biomimetic:CAP0402-CAP
- C30: value 12pF -> 22uF; device SparkFun:CAP0402-CAP -> biomimetic:CAP0603-CAP
- C31: device SparkFun:CAP0402-CAP -> biomimetic:CAP0402-CAP; DIELECTRIC (none) -> X7R; TECHNOLOGY (none) -> CERAMIC; VOLTAGE (none) -> 16V
- C4, C5, C7: value 0.1uF -> 1uF; device SparkFun:CAP0402-CAP -> biomimetic:CAP0402-CAP
- C6: value 10nF -> 0.1uF; device SparkFun:CAP0402-CAP -> biomimetic:CAP0402-CAP
- C8: value 2.2uF -> 1uF; device SparkFun:CAP0402-CAP -> biomimetic:CAP0402-CAP
- JP2: value MPCS2PH -> MOLEX_503480-0600; device stan:MPCS2PH -> biomimetic:MOLEX_503480-0600
- JP3: value 51441-2493-C -> MOLEX_503480-0600; device stan:OV7660FSL_CON-24 -> biomimetic:MOLEX_503480-0600
- R1: value 4.7k -> 1k; device rcl:R-US_R0402 -> biomimetic:RESISTOR0402-RES
- R10: value 10k -> 47k; device rcl:R-US_R0402 -> biomimetic:RESISTOR0402-RES; TOLERANCE (none) -> 1%
- R11: value 470 -> 15k; device rcl:R-US_R0402 -> biomimetic:RESISTOR0402-RES; TOLERANCE (none) -> 1%
- R13: value 470 -> 47k; device rcl:R-US_R0402 -> biomimetic:RESISTOR0402-RES; TOLERANCE (none) -> 1%
- R16: value 27K -> 4.7k; device rcl:R-US_R0402 -> biomimetic:RESISTOR0402-RES; TOLERANCE (none) -> 1%
- R17: value 10K -> 15k; device rcl:R-US_R0402 -> biomimetic:RESISTOR0402-RES; TOLERANCE (none) -> 1%
- R18: value 470 -> 4.7k; device rcl:R-US_R0402 -> biomimetic:RESISTOR0402-RES; TOLERANCE (none) -> 1%
- R2: value 4.7k -> 2.7k; device rcl:R-US_R0402 -> biomimetic:RESISTOR0402-RES
- R3, R4: device rcl:R-US_R0402 -> biomimetic:RESISTOR0402-RES
Connections:
- removed net AN0: C31.2, PROC1.RB0/AN0, R16.2, R17.1
- removed net AN1: PROC1.RB1/AN1
- removed net AN10: PROC1.RB10/AN10/TMS
- removed net AN11: PROC1.RB11/AN11/TDO
- removed net AN3: PROC1.RB3/AN3
- removed net AN4: PROC1.RB4/AN4
- removed net AN5: PROC1.RB5/AN5
- removed net BAT+: C15.1, C24.1, JP2.1, R17.2, U1.EN1, U1.EN2, U1.VIN, U2.EN1, U2.EN2, U2.VIN, U9.VDD
- removed net INT1: PROC1.RD8/IC1/INT1/FLTA, U4.INT
- removed net INT2: PROC1.RD9/IC2/INT2/FLTB/U1CTS, U9.OUT
- removed net INT3: PROC1.RD10/IC3/INT3
- removed net INT4: PROC1.RD11/IC4/INT4, U8.IRQ
- removed net MCLR: J2.5, PROC1.MCLR, R10.1
- removed net OSC1: JP3.XCLK, PROC1.RC12/CLKI/OSC1, U6.OUT
- removed net OSC2: PROC1.RC15/CLKO/OSC2
- removed net PWM1: PROC1.PWM1L/RE0
- removed net PWM1H: PROC1.PWM1H/RE1
- removed net PWM2: PROC1.PWM2L/RE2
- removed net PWM2H: PROC1.PWM2H/RE3
- removed net PWM3: PROC1.PWM3L/RE4
- removed net PWM3H: PROC1.PWM3H/RE5
- removed net PWM4: PROC1.PWM4L/RE6
- removed net PWM4H: PROC1.PWM4H/RE7
- removed net RB15: PROC1.RB15/AN15/CN12/OCFB, U8.SLP_TR
- removed net RC13: JP3.VSYNC, PROC1.T4CK/CN1/RC13
- removed net RC14: JP3.PWDN, PROC1.T1CK/CN0/RC14
- removed net RD0: PROC1.RD0/OC1
- removed net RD1: PROC1.RD1
- removed net RD10: JP3.D0
- removed net RD11: JP3.D4
- removed net RD12: JP3.D5
- removed net RD13: JP3.D6
- removed net RD14: JP3.D7
- removed net RD15: JP3.D1
- removed net RD2: PROC1.RD2
- removed net RD3: PROC1.RD3
- removed net RD4: PROC1.RD4
- removed net RD5: PROC1.RD5
- removed net RD6: PROC1.RD6
- removed net RD7: PROC1.RD7
- removed net RD8: JP3.D2
- removed net RD9: JP3.D3
- removed net RF0: JP3.HREF, PROC1.RF0
- removed net RF1: JP3.PCLK, PROC1.RF1
- removed net SCL2: PROC1.SCL2/U2TX/RF5, R4.1, U4.SCL
- removed net SDA2: PROC1.SDA2/U2RX/RF4, R3.1, U4.SDA
- removed net SS1: PROC1.RB2/AN2, U8./SEL
- removed net SS2: PROC1.SS2/CN11/RG9, U3./CS
- removed net VCC: C17.1, C3.2, JP3.AVDD, JP3.DOVDD, U2.VOUT1
- removed net VDD: C12.1, C2.1, C23.1, C25.1, C4.1, C6.1, C7.1, J2.4, PROC1.AVDD, PROC1.VDD@10, PROC1.VDD@26, PROC1.VDD@38, PROC1.VDD@57, R1.2, R10.2, R2.2, R3.2, R4.2, U1.VOUT1, U3./RESET, U3./WP, U3.VCC, U4.VDD, U4.VLOGIC, U6.VDD, U8./RST, U8.DEVDD, U8.EVDD
- removed net VEE: C16.1, JP3.DVDD, U2.VOUT2
- removed net VPP: C26.1, U1.VOUT2
- new net !RESET: IC10S.!RESET, IC4RESET/CLOCK/DEBUG.!MCLR, IC5S.!RST, JP1.1, R3.1
- new net !SS1: IC4SERIAL.AN2/!SS1!/CN4/RB2, IC5S.!SEL
- new net !SS2_1: IC10S.!CS, IC4SERIAL.!SS2!/CN11/RG9
- new net !SS2_2: IC4SERIAL.OSC2/CLKO/RC15, IC9S.!CS
- new net 1.8V: C8.1, IC3.1.8V, JP4.DVDD
- new net 2.5V: C2.1, C36.2, IC3.2.5V, JP4.AVDD, JP4.DOVDD
- new net 3.0V: C7.1, IC2.3.0
- new net 3.3V: C1.1, C11.1, C12.1, C13.1, C14.1, C21.1, C23.1, C37.1, C40.1, C9.1, IC10P.V+, IC10S.!WP, IC2.3.3V, IC4P_VDD@10.V+, IC4P_VDD@26.V+, IC4P_VDD@38.V+, IC4P_VDD@57.V+, IC5P_DEVDD.V+, IC5P_EVDD.V+, IC9P_VDD.V+, JP1.2, JP3.1, L1.2, OSC1.VDD, R3.2, R4.2, R5.2
- new net 40MHZ: IC4RESET/CLOCK/DEBUG.OSC1/CLKIN/RC12, JP4.XCLK, OSC1.OUT
- new net BATT_LEVEL: C6.1, IC4ANALOG.PGED3/AN0/VREF+/CN2/RB0, R1.1, R2.2
- new net CAM_D0: IC4GPIO.OC1/RD0, JP4.D0
- new net CAM_D1: IC4GPIO.OC2/RD1, JP4.D1
- new net CAM_D2: IC4GPIO.OC3/RD2, JP4.D2
- new net CAM_D3: IC4GPIO.OC4/RD3, JP4.D3
- new net CAM_D4: IC4GPIO.OC5/IC5/CN13/RD4, JP4.D4
- new net CAM_D5: IC4GPIO.OC6/IC6/CN14/RD5, JP4.D5
- new net CAM_D6: IC4GPIO.OC7/CN15/RD6, JP4.D6
- new net CAM_D7: IC4GPIO.OC8/UPDN/CN16/RD7, JP4.D7
- new net CAM_HREF: IC4GPIO.C1RX/RF0, IC9S.FSYNC, JP4.HREF
- new net CAM_PCLK: IC4GPIO.C1TX/RF1, JP4.PCLK
- new net CAM_PWDN: IC4GPIO.PGEC2/SOSCO/T1CK/CN0/RC14, JP4.PWDN
- new net CAM_VSYNC: IC4GPIO.PGED2/SOSCI/T4CK/CN1/RC13, JP4.VSYNC
- new net EXT1: IC4GPIO.PGEC3/AN1/VREF-/CN3/RB1, P11.P
- new net EXT2: IC4GPIO.AN3/INDX/CN5/RB3, P12.P
- new net EXT3: IC4GPIO.AN4/QEA/IC7/CN6/RB4, P13.P
- new net EXT4: IC4GPIO.AN5/QEB/IC8/CN7/RB5, P14.P
- new net EXT5: IC4GPIO.IC1/!FLTA!/INT1/RD8, P15.P
- new net EXT6: IC4GPIO.IC3/INT3/RD10, P16.P
- new net GN_LED: IC4GPIO.TDI/AN13/RB13, LED2.A
- new net LOWBATT_IRQ: IC1.VOUT, IC4GPIO.IC2/!U1CTS!/!FLTB!/INT2/RD9
- new net MOTOR_A_BEMF: IC4ANALOG.!U2CTS!/AN8/RB8, IC6A.OUT, R8.2
- new net MOTOR_A_IN1: IC4PWM.PWM1H/RE1, IC7S.AIN1
- new net MOTOR_A_IN2: IC4PWM.PWM1L/RE0, IC7S.AIN2
- new net MOTOR_A_OUT1: C24.1, IC7S.AOUT1, P3.P, R9.1
- new net MOTOR_A_OUT2: C24.2, IC7S.AOUT2, P4.P, R10.1
- new net MOTOR_B_BEMF: IC4ANALOG.AN9/RB9, IC6B.OUT, R12.2
- new net MOTOR_B_IN1: IC4PWM.PWM2H/RE3, IC7S.BIN1
- new net MOTOR_B_IN2: IC4PWM.PWM2L/RE2, IC7S.BIN2
- new net MOTOR_B_OUT1: C25.1, IC7S.BOUT1, P5.P, R13.1
- new net MOTOR_B_OUT2: C25.2, IC7S.BOUT2, P6.P, R14.1
- new net MOTOR_C_BEMF: IC4ANALOG.TMS/AN10/RB10, IC6C.OUT, R17.2
- new net MOTOR_C_IN1: IC4PWM.PWM3H/RE5, IC8S.AIN1
- new net MOTOR_C_IN2: IC4PWM.PWM3L/RE4, IC8S.AIN2
- new net MOTOR_C_OUT1: C27.1, IC8S.AOUT1, P7.P, R19.1
- new net MOTOR_C_OUT2: C27.2, IC8S.AOUT2, P8.P, R20.1
- new net MOTOR_D_BEMF: IC4ANALOG.TDO/AN11/RB11, IC6D.OUT, R22.2
- new net MOTOR_D_IN1: IC4PWM.PWM4H/RE7, IC8S.BIN1
- new net MOTOR_D_IN2: IC4PWM.PWM4L/RE6, IC8S.BIN2
- new net MOTOR_D_OUT1: C28.1, IC8S.BOUT1, P9.P, R23.1
- new net MOTOR_D_OUT2: C28.2, IC8S.BOUT2, P10.P, R24.1
- new net N$1: C22.2, IC5P_DVDD.V+
- new net N$11: LED_RX.C, R7.1
- new net N$21: C10.1, IC4P_AVDD.V+, L1.1
- new net N$24: IC6C.-IN, R17.1, R19.2
- new net N$3: C20.2, IC5P_AVDD.V+
- new net N$31: IC6A.+IN, R10.2, R11.2
- new net N$32: C39.2, IC9P_REGOUT.V-
- new net N$6: C16.1, IC5S.RFP
- new net N$7: C17.2, IC5S.RFN
- new net N$8: C19.1, IC5S.XTAL2, OSC2.OUT/IN
- new net N$9: C18.1, IC5S.XTAL1, OSC2.IN/OUT
- new net PGC: IC4RESET/CLOCK/DEBUG.PGEC1/AN6/OCFA/RB6, JP1.5
- new net PGD: IC4RESET/CLOCK/DEBUG.PGED1/AN7/RB7, JP1.4
- new net RADIO_IRQ: IC4GPIO.IC4/INT4/RD11, IC5S.IRQ
- new net RADIO_SLP_TR: IC4GPIO.AN15/OCFB/CN12/RB15, IC5S.SLP_TR
- new net RD_LED: IC4GPIO.TCK/AN12/RB12, LED3.A
- new net U2RX: IC4SERIAL.U2RX/SDA2/CN17/RF4, JP2.6
- new net U2TX: IC4SERIAL.U2TX/SCL2/CN18/RF5, JP2.4
- new net V_BATT: C29.1, C3.1, C30.1, C31.1, C33.1, C34.1, C4.2, C5.2, IC1.VIN, IC2.EN_3.0V, IC2.EN_3.3V, IC2.VIN, IC3.EN_1.8V, IC3.EN_2.5V, IC3.VIN, IC6P.V+, IC7P_VM.V+, IC7S.!SLEEP, IC8P_VM.V+, IC8S.!SLEEP, JP2.1, JP2.2, P1.P, R1.2, R16.2
- new net V_REF: C26.1, R11.1, R15.1, R16.1, R18.2, R21.1, R25.1
- new net YW_LED: IC4GPIO.!U2RTS!/AN14/RB14, LED1.A
- net GND: now also B1.GND, B1.RFGND, C1.2, C10.2, C14.2, C18.2, C19.2, C20.1, C21.2, C22.1, C3.2, C32.2, C33.2, C35.2, C36.1, C37.2, C38.1, C39.1, C4.1, C40.2, C5.1, C9.2, IC1.VSS, IC10P.V-, IC2.GND, IC3.GND, IC4P_AVDD.V-, IC4P_VDD@10.V-, IC4P_VDD@26.V-, IC4P_VDD@38.V-, IC5P_AVSS.V-, IC5P_DVSS.V-, IC6P.V-, IC7P_VM.V-, IC7S.AISEN, IC7S.BISEN, IC8P_VM.V-, IC8S.AISEN, IC8S.BISEN, IC9P_VDD.V-, IC9S.CLKIN, JP1.3, JP2.3, JP2.5, JP3.2, JP3.4, JP3.6, JP4.AGND, JP4.DGND, JP4.RESET, OSC1.GND, OSC2.GND, OSC2.GND@2, P2.P, R18.1, R2.1, R26.2, R27.2, R28.2, R6.2, R7.2; no longer BALUN1.GND, BALUN1.NC, BALUN1.RFGND, C1.1, C16.2, C17.2, C24.2, C25.2, C3.1, C31.1, C4.2, C5.2, J2.3, JP2.2, JP3.AGND, JP3.DGND, JP3.RESET, PROC1.AVSS, PROC1.VSS@25, PROC1.VSS@41, PROC1.VSS@9, R11.2, R13.2, R16.1, R18.2, U1.GND, U2.GND, U3.GND, U4.AD0, U4.CLKIN, U4.GND, U4.RESV-G, U6.GND, U7.GND, U7.GND@2, U8.AVSS, U8.AVSS@27, U8.AVSS@30, U8.AVSS@31, U8.AVSS@32, U8.AVSS@6, U8.DVSS, U8.DVSS@12, U8.DVSS@16, U8.DVSS@18, U8.DVSS@21, U8.GDNPAD, U9.VSS
- net N$10: now also B1.BAL3, C17.1; no longer BALUN1.BAL4, C14.1
- net N$12: now also B1.BAL4, C16.2; no longer BALUN1.BAL3, C28.1
- net N$13: now also IC5S.DIG3, LED_RX.A; no longer C14.2, U8.RFP
- net N$14: now also IC5S.DIG2, LED_TX.A; no longer C28.2, U8.RFN
- net N$15: now also LED1.C, R26.1; no longer BALUN1.UNBAL, U11.SIGNAL
- net N$16: now also LED2.C, R27.1; no longer C30.1, U7.IN/OUT@2, U8.XTAL2
- net N$17: now also LED3.C, R28.1; no longer C29.1, U7.IN/OUT, U8.XTAL1
- net N$18: now also C32.1, IC7P_VINT.V-; no longer C1.2, U4.CPOUT
- net N$19: now also C34.2, IC8P_VCP.V+; no longer C5.1, U4.REGOUT
- net N$2: now also C31.2, IC7P_VCP.V+; no longer J2.6, PROC1.RB8/AN8/U2CTS
- net N$20: now also C35.1, IC8P_VINT.V-; no longer LED4.C, R11.1
- net N$22: now also IC6B.-IN, R12.1, R13.2; no longer LED4.A, PROC1.RB14/AN14/U2RTS
- net N$23: now also IC6B.+IN, R14.2, R15.2; no longer J2.1, PROC1.RB6/AN6/PGC1
- net N$25: now also IC6C.+IN, R20.2, R21.2; no longer J2.2, PROC1.RB7/AN7/PGD1
- net N$26: now also IC6D.-IN, R22.1, R23.2; no longer LED5.C, R13.1
- net N$27: now also IC6D.+IN, R24.2, R25.2; no longer LED6.C, R18.1
- net N$28: now also C15.1, IC4P_VCAP.V+; no longer LED5.A, PROC1.RB13/AN13/TDI
- net N$29: now also C38.2, IC9P_CPOUT.V-; no longer LED6.A, PROC1.RB12/AN12/TCK
- net N$30: now also IC6A.-IN, R8.1, R9.2; no longer C8.1, PROC1.VCAP
- net N$4: now also ANT1.SIGNAL, B1.UNBAL; no longer C11.1, U8.AVDD
- net N$5: now also LED_TX.C, R6.1; no longer C13.1, U8.DVDD@13, U8.DVDD@14
- net SCK1: now also IC4SERIAL.!U1RTS!/SCK1/INT0/RF6, IC5S.SCLK; no longer PROC1.INT0/U1RTS/SCK1/RF6, U8.SCLK
- net SCK2: now also IC10S.SCK, IC4SERIAL.SCK2/CN8/RG6, IC9S.SCL/SCLK; no longer PROC1.SCK2/CN8/RG6, U3.SCK
- net SCL1: now also IC4SERIAL.SCL1/RG2, JP3.3, JP4.SIO_C, R4.1; no longer JP3.SIO_C, PROC1.SCL1, R1.1
- net SDA1: now also IC4SERIAL.SDA1/RG3, JP3.5, JP4.SIO_D, R5.1; no longer JP3.SIO_D, PROC1.SDA1, R2.1
- net SDI1: now also IC4SERIAL.U1RX/SDI1/RF2, IC5S.MISO; no longer PROC1.SDI1/U1RX/RF2, U8.MISO
- net SDI2: now also IC10S.SO, IC4SERIAL.SDI2/CN9/RG7, IC9S.AD0/SDO; no longer PROC1.SDI2/CN9/RG7, U3.SO
- net SDO1: now also IC4SERIAL.U1TX/SDO1/RF3, IC5S.MOSI; no longer PROC1.SDO1/U1TX/RF3, U8.MOSI
- net SDO2: now also IC10S.SI, IC4SERIAL.SDO2/CN10/RG8, IC9S.SDA/SDI; no longer PROC1.SDO2/CN10/RG8, U3.SI
Other:
- note removed: "1.8V"
- note removed: "2.5V"
- note removed: "3.0V"
- note removed: "3.3V"

Commit message: Work 6/30
Connections:
- net 3.3V: now also C29.1, IC6P.V+
- net V_BATT: no longer C29.1, IC6P.V+
Changed lines of the file:
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@@
 <wire x1="170.18" y1="167.64" x2="170.18" y2="177.8" width="0.1524" layer="91"/>
 <wire x1="170.18" y1="177.8" x2="165.1" y2="177.8" width="0.1524" layer="91"/>
-<label x="175.26" y="167.64" size="1.778" layer="95"/>
+<label x="205.74" y="167.64" size="1.778" layer="95"/>
 <pinref part="IC6" gate="A" pin="OUT"/>
 <wire x1="167.64" y1="167.64" x2="170.18" y2="167.64" width="0.1524" layer="91"/>
@@
 <net name="V_BATT" class="0">
 <segment>
-<pinref part="U$3" gate="G$1" pin="3.3V"/>
-<pinref part="IC6" gate="P" pin="V+"/>
-<wire x1="121.92" y1="30.48" x2="121.92" y2="27.94" width="0.1524" layer="91"/>
-<pinref part="C29" gate="G$1" pin="1"/>
-<wire x1="121.92" y1="27.94" x2="121.92" y2="25.4" width="0.1524" layer="91"/>
-<wire x1="127" y1="22.86" x2="127" y2="27.94" width="0.1524" layer="91"/>
-<wire x1="127" y1="27.94" x2="121.92" y2="27.94" width="0.1524" layer="91"/>
-<junction x="121.92" y="27.94"/>
-</segment>
-<segment>
 <pinref part="U$14" gate="G$1" pin="V_BATT"/>
 <pinref part="IC8" gate="P_VM" pin="V+"/>
@@
 </segment>
 </net>
+<net name="3.3V" class="0">
+<segment>
+<pinref part="U$3" gate="G$1" pin="3.3V"/>
+<pinref part="IC6" gate="P" pin="V+"/>
+<wire x1="121.92" y1="30.48" x2="121.92" y2="27.94" width="0.1524" layer="91"/>
+<pinref part="C29" gate="G$1" pin="1"/>
+<wire x1="121.92" y1="27.94" x2="121.92" y2="25.4" width="0.1524" layer="91"/>
+<wire x1="121.92" y1="27.94" x2="127" y2="27.94" width="0.1524" layer="91"/>
+<wire x1="127" y1="27.94" x2="127" y2="22.86" width="0.1524" layer="91"/>
+<junction x="121.92" y="27.94"/>
+</segment>
+</net>

Commit message: Commit before replace LTC6088 with LT1991
Parts:
- added C41, C42, C44: (no value), biomimetic:CAP0402-CAP
- added C43: xnF, biomimetic:CAP0402-CAP
- added R29, R30, R31, R32: (no value), biomimetic:RESISTOR0402-RES
Connections:
- new net N$34: IC6D.OUT, R22.2, R32.1
- new net N$35: IC6C.OUT, R17.2, R31.1
- new net N$36: IC6A.OUT, R29.1, R8.2
- new net N$37: IC6B.OUT, R12.2, R30.1
- net GND: now also C41.2, C42.2, C43.2, C44.2
- net MOTOR_A_BEMF: now also C41.1, R29.2; no longer IC6A.OUT, R8.2
- net MOTOR_B_BEMF: now also C42.1, R30.2; no longer IC6B.OUT, R12.2
- net MOTOR_C_BEMF: now also C43.1, R31.2; no longer IC6C.OUT, R17.2
- net MOTOR_D_BEMF: now also C44.1, R32.2; no longer IC6D.OUT, R22.2
Other:
- moved on the sheet: C26, IC6A, IC6B, IC6C, IC6D, R10, R11, R12, R13, R14, R15, R16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

Commit message: RF top layout complete
Connections:
- net CAM_D5 renamed N#3
Changed lines of the file:
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@@
 <class number="0" name="default" width="0" drill="0">
-</class>
-<class number="1" name="sup" width="0.254" drill="0">
 </class>
 </classes>
@@
 </busses>
 <nets>
-<net name="GND" class="1">
+<net name="GND" class="0">
 <segment>
 <pinref part="R2" gate="G$1" pin="1"/>
@@
 </busses>
 <nets>
-<net name="GND" class="1">
+<net name="GND" class="0">
 <segment>
 <wire x1="76.2" y1="71.12" x2="81.28" y2="71.12" width="0.1524" layer="91"/>
@@
 </segment>
 </net>
-<net name="CAM_D5" class="0">
+<net name="N#3" class="0">
 <segment>
 <wire x1="99.06" y1="127" x2="96.52" y2="127" width="0.1524" layer="91"/>
@@
 </busses>
 <nets>
-<net name="GND" class="1">
+<net name="GND" class="0">
 <segment>
 <pinref part="GND17" gate="1" pin="GND"/>
@@
 </busses>
 <nets>
-<net name="GND" class="1">
+<net name="GND" class="0">
 <segment>
 <wire x1="66.04" y1="147.32" x2="68.58" y2="147.32" width="0.1524" layer="91"/>
@@
 </busses>
 <nets>
-<net name="GND" class="1">
+<net name="GND" class="0">
 <segment>
 <wire x1="114.3" y1="154.94" x2="114.3" y2="165.1" width="0.1524" layer="91"/>
@@
 </segment>
 </net>
-<net name="CAM_D5" class="0">
+<net name="N#3" class="0">
 <segment>
 <pinref part="JP4" gate="G$1" pin="D5"/>

Commit message: Partial IMU/flash route. PIC, IMU, and flash locations locked. Passives for IMU/flash.
Parts:
- removed P15: EXT5, wirepad:SMD2
Connections:
- removed net EXT5: IC4GPIO.IC1/!FLTA!/INT1/RD8, P15.P
- new net CAM_D5: IC4GPIO.OC6/IC6/CN14/RD5
- new net IMU_IRQ: IC4GPIO.IC1/!FLTA!/INT1/RD8, IC9S.INT
- net N#3: no longer IC4GPIO.OC6/IC6/CN14/RD5
Other:
- moved on the sheet: P16
Changed lines of the file:
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@@
 <part name="P13" library="wirepad" deviceset="SMD2" device="" value="EXT3"/>
 <part name="P14" library="wirepad" deviceset="SMD2" device="" value="EXT4"/>
-<part name="P15" library="wirepad" deviceset="SMD2" device="" value="EXT5"/>
 <part name="P16" library="wirepad" deviceset="SMD2" device="" value="EXT6"/>
 <part name="C41" library="biomimetic" deviceset="CAP" device="0402-CAP"/>
@@
 </segment>
 </net>
-<net name="N#3" class="0">
-<segment>
-<wire x1="99.06" y1="127" x2="96.52" y2="127" width="0.1524" layer="91"/>
-<label x="101.6" y="127" size="1.778" layer="95"/>
-<pinref part="IC4" gate="GPIO" pin="OC6/IC6/CN14/RD5"/>
-</segment>
-</net>
 <net name="CAM_D6" class="0">
 <segment>
@@
 <wire x1="35.56" y1="124.46" x2="33.02" y2="124.46" width="0.1524" layer="91"/>
 <label x="12.7" y="124.46" size="1.778" layer="95"/>
-</segment>
-</net>
-<net name="EXT5" class="0">
-<segment>
-<pinref part="IC4" gate="GPIO" pin="IC1/!FLTA!/INT1/RD8"/>
-<wire x1="96.52" y1="119.38" x2="99.06" y2="119.38" width="0.1524" layer="91"/>
-<label x="101.6" y="119.38" size="1.778" layer="95"/>
 </segment>
 </net>
@@
 <pinref part="IC4" gate="P_VCAP" pin="V+"/>
 <wire x1="111.76" y1="17.78" x2="111.76" y2="22.86" width="0.1524" layer="91"/>
+</segment>
+</net>
+<net name="CAM_D5" class="0">
+<segment>
+<wire x1="99.06" y1="127" x2="96.52" y2="127" width="0.1524" layer="91"/>
+<label x="101.6" y="127" size="1.778" layer="95"/>
+<pinref part="IC4" gate="GPIO" pin="OC6/IC6/CN14/RD5"/>
+</segment>
+</net>
+<net name="IMU_IRQ" class="0">
+<segment>
+<pinref part="IC4" gate="GPIO" pin="IC1/!FLTA!/INT1/RD8"/>
+<wire x1="96.52" y1="119.38" x2="99.06" y2="119.38" width="0.1524" layer="91"/>
+<label x="101.6" y="119.38" size="1.778" layer="95"/>
 </segment>
 </net>
@@
 <attribute name="VALUE" x="218.44" y="162.56" size="1.778" layer="96"/>
 </instance>
-<instance part="P15" gate="1" x="228.6" y="160.02" smashed="yes">
+<instance part="P16" gate="1" x="228.6" y="160.02" smashed="yes">
 <attribute name="NAME" x="210.82" y="160.02" size="1.778" layer="95"/>
 <attribute name="VALUE" x="218.44" y="160.02" size="1.778" layer="96"/>
-</instance>
-<instance part="P16" gate="1" x="228.6" y="157.48" smashed="yes">
-<attribute name="NAME" x="210.82" y="157.48" size="1.778" layer="95"/>
-<attribute name="VALUE" x="218.44" y="157.48" size="1.778" layer="96"/>
 </instance>
 </instances>
@@
 </segment>
 </net>
-<net name="EXT5" class="0">
-<segment>
-<pinref part="P15" gate="1" pin="P"/>
+<net name="EXT6" class="0">
+<segment>
+<pinref part="P16" gate="1" pin="P"/>
 <wire x1="231.14" y1="160.02" x2="233.68" y2="160.02" width="0.1524" layer="91"/>
 <label x="236.22" y="160.02" size="1.778" layer="95"/>
-</segment>
-</net>
-<net name="EXT6" class="0">
-<segment>
-<pinref part="P16" gate="1" pin="P"/>
-<wire x1="231.14" y1="157.48" x2="233.68" y2="157.48" width="0.1524" layer="91"/>
-<label x="236.22" y="157.48" size="1.778" layer="95"/>
 </segment>
 </net>
@@
 </segment>
 </net>
+<net name="IMU_IRQ" class="0">
+<segment>
+<pinref part="IC9" gate="S" pin="INT"/>
+<wire x1="63.5" y1="76.2" x2="66.04" y2="76.2" width="0.1524" layer="91"/>
+<label x="68.58" y="76.2" size="1.778" layer="95"/>
+</segment>
+</net>
