File: ImageProc.sch (EAGLE design)
At the start: 117 parts, among them IC1 XC61GC3002HR-G, IC10 AT45DB642D-CNU, IC2 MIC5335-SPYMT, IC3 MIC5335-JGYMT, IC4 DSPIC33FJ128MC706A, IC5 AT86RF233-ZU, IC6 LTC6088, IC7 DRV8833RTY, IC8 DRV8833RTY, IC9 MPU-6000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

Commit message: Added sheet name headings
Other:
- moved on the sheet: 3.3V, C36, C9, GND, IC10S, IC4ANALOG, IC4GPIO, IC4PWM, IC4RESET/CLOCK/DEBUG, IC4SERIAL, IC9S, JP1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

Commit message: Resolved the three wiring issues (non-connect on the v_batt plane, non-connect for a logic ground, and programming connector backwards).
Added the biomimetics dru's
Connections:
- net !RESET: now also JP1.5; no longer JP1.1
- net 3.3V: now also JP1.4; no longer JP1.2
- net PGC: now also JP1.1; no longer JP1.5
- net PGD: now also JP1.2; no longer JP1.4
Changed lines of the file:
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@@
 <part name="GND4" library="biomimetic" deviceset="GND" device=""/>
 <part name="P+12" library="biomimetic" deviceset="3.3V" device=""/>
-<part name="GND37" library="supply1" deviceset="GND" device=""/>
-<part name="P+14" library="biomimetic" deviceset="3.3V" device=""/>
 <part name="P+19" library="biomimetic" deviceset="3.3V" device=""/>
 <part name="GND43" library="supply1" deviceset="GND" device=""/>
@@
 <instance part="R27" gate="G$1" x="50.8" y="119.38"/>
 <instance part="R28" gate="G$1" x="50.8" y="109.22"/>
-<instance part="GND37" gate="1" x="114.3" y="142.24"/>
-<instance part="P+14" gate="G$1" x="114.3" y="167.64"/>
 <instance part="P+7" gate="G$1" x="71.12" y="30.48"/>
 <instance part="C40" gate="G$1" x="76.2" y="20.32"/>
@@
 <nets>
 <net name="GND" class="0">
-<segment>
-<wire x1="114.3" y1="144.78" x2="114.3" y2="154.94" width="0.1524" layer="91"/>
-<wire x1="114.3" y1="154.94" x2="109.22" y2="154.94" width="0.1524" layer="91"/>
-<pinref part="GND37" gate="1" pin="GND"/>
-<label x="116.84" y="154.94" size="1.778" layer="95"/>
-<pinref part="JP1" gate="G$1" pin="3"/>
-</segment>
 <segment>
 <pinref part="GND41" gate="1" pin="GND"/>
@@
 <wire x1="218.44" y1="147.32" x2="218.44" y2="144.78" width="0.1524" layer="91"/>
 </segment>
+<segment>
+<pinref part="JP1" gate="G$1" pin="3"/>
+<wire x1="109.22" y1="154.94" x2="121.92" y2="154.94" width="0.1524" layer="91"/>
+<label x="127" y="154.94" size="1.778" layer="95"/>
+</segment>
 </net>
 <net name="CAM_PCLK" class="0">
@@
 <net name="!RESET" class="0">
 <segment>
-<label x="116.84" y="160.02" size="1.778" layer="95"/>
-<wire x1="109.22" y1="160.02" x2="111.76" y2="160.02" width="0.1524" layer="91"/>
-<pinref part="JP1" gate="G$1" pin="1"/>
-</segment>
-<segment>
 <wire x1="104.14" y1="73.66" x2="101.6" y2="73.66" width="0.1524" layer="91"/>
 <label x="91.44" y="73.66" size="1.778" layer="95"/>
 <pinref part="IC10" gate="S" pin="!RESET"/>
 </segment>
+<segment>
+<pinref part="JP1" gate="G$1" pin="5"/>
+<wire x1="109.22" y1="149.86" x2="121.92" y2="149.86" width="0.1524" layer="91"/>
+<label x="127" y="149.86" size="1.778" layer="95"/>
+</segment>
 </net>
 <net name="3.3V" class="0">
-<segment>
-<wire x1="109.22" y1="157.48" x2="114.3" y2="157.48" width="0.1524" layer="91"/>
-<wire x1="114.3" y1="157.48" x2="114.3" y2="167.64" width="0.1524" layer="91"/>
-<pinref part="P+14" gate="G$1" pin="3.3V"/>
-<label x="116.84" y="157.48" size="1.778" layer="95"/>
-<pinref part="JP1" gate="G$1" pin="2"/>
-</segment>
 <segment>
 <wire x1="104.14" y1="78.74" x2="101.6" y2="78.74" width="0.1524" layer="91"/>
@@
 <wire x1="218.44" y1="162.56" x2="218.44" y2="165.1" width="0.1524" layer="91"/>
 </segment>
+<segment>
+<pinref part="JP1" gate="G$1" pin="4"/>
+<wire x1="109.22" y1="152.4" x2="121.92" y2="152.4" width="0.1524" layer="91"/>
+<label x="127" y="152.4" size="1.778" layer="95"/>
+</segment>
 </net>
 <net name="40MHZ" class="0">
@@
 <label x="198.12" y="96.52" size="1.778" layer="95"/>
 <pinref part="JP4" gate="G$1" pin="XCLK"/>
-</segment>
-</net>
-<net name="PGD" class="0">
-<segment>
-<label x="116.84" y="152.4" size="1.778" layer="95"/>
-<wire x1="109.22" y1="152.4" x2="111.76" y2="152.4" width="0.1524" layer="91"/>
-<pinref part="JP1" gate="G$1" pin="4"/>
-</segment>
-</net>
-<net name="PGC" class="0">
-<segment>
-<label x="116.84" y="149.86" size="1.778" layer="95"/>
-<wire x1="109.22" y1="149.86" x2="111.76" y2="149.86" width="0.1524" layer="91"/>
-<pinref part="JP1" gate="G$1" pin="5"/>
 </segment>
 </net>
@@
 </segment>
 </net>
+<net name="PGC" class="0">
+<segment>
+<pinref part="JP1" gate="G$1" pin="1"/>
+<wire x1="109.22" y1="160.02" x2="121.92" y2="160.02" width="0.1524" layer="91"/>
+<label x="127" y="160.02" size="1.778" layer="95"/>
+</segment>
+</net>
+<net name="PGD" class="0">
+<segment>
+<pinref part="JP1" gate="G$1" pin="2"/>
+<wire x1="109.22" y1="157.48" x2="121.92" y2="157.48" width="0.1524" layer="91"/>
+<label x="127" y="157.48" size="1.778" layer="95"/>
+</segment>
+</net>
